Commit message: fix gripper TF

File: urdf/Dual_piper_ROS2.xacro (robot description, xacro)
@@ -171,5 +171,5 @@
   </inertial>
   <visual>
-    <origin xyz="0.438169 -0.790481 0.810851" rpy="0 0 0"/>
+    <origin xyz="${-0.22209+0.438169} ${0.395033-0.790481} ${-0.406013+0.810851}" rpy="0 0 0"/>
     <geometry>
       <mesh filename="file://$(find Dual_piper_ROS2_description)/meshes/piper_right_L_1.stl" scale="0.001 0.001 0.001"/>
@@ -178,5 +178,5 @@
   </visual>
   <collision>
-    <origin xyz="0.438169 -0.790481 0.810851" rpy="0 0 0"/>
+    <origin xyz="${-0.22209+0.438169} ${0.395033-0.790481} ${-0.406013+0.810851}" rpy="0 0 0"/>
     <geometry>
       <mesh filename="file://$(find Dual_piper_ROS2_description)/meshes/piper_right_L_1.stl" scale="0.001 0.001 0.001"/>
@@ -191,5 +191,5 @@
   </inertial>
   <visual>
-    <origin xyz="0.438169 -0.790481 0.810851" rpy="0 0 0"/>
+    <origin xyz="${-0.22209+0.438169} ${0.395033-0.790481} ${-0.406013+0.810851}" rpy="0 0 0"/>
     <geometry>
       <mesh filename="file://$(find Dual_piper_ROS2_description)/meshes/piper_left_L_1.stl" scale="0.001 0.001 0.001"/>
@@ -198,5 +198,5 @@
   </visual>
   <collision>
-    <origin xyz="0.438169 -0.790481 0.810851" rpy="0 0 0"/>
+    <origin xyz="${-0.22209+0.438169} ${0.395033-0.790481} ${-0.406013+0.810851}" rpy="0 0 0"/>
     <geometry>
       <mesh filename="file://$(find Dual_piper_ROS2_description)/meshes/piper_left_L_1.stl" scale="0.001 0.001 0.001"/>
@@ -351,5 +351,5 @@
   </inertial>
   <visual>
-    <origin xyz="-0.358864 -0.806368 0.810912" rpy="0 0 0"/>
+    <origin xyz="${0.176294-0.358864} ${0.41092-0.806368} ${-0.406074+0.810912}" rpy="0 0 0"/>
     <geometry>
       <mesh filename="file://$(find Dual_piper_ROS2_description)/meshes/piper_left_R_1.stl" scale="0.001 0.001 0.001"/>
@@ -358,5 +358,5 @@
   </visual>
   <collision>
-    <origin xyz="-0.358864 -0.806368 0.810912" rpy="0 0 0"/>
+    <origin xyz="${0.176294-0.358864} ${0.41092-0.806368} ${-0.406074+0.810912}" rpy="0 0 0"/>
     <geometry>
       <mesh filename="file://$(find Dual_piper_ROS2_description)/meshes/piper_left_R_1.stl" scale="0.001 0.001 0.001"/>
@@ -371,5 +371,5 @@
   </inertial>
   <visual>
-    <origin xyz="-0.358864 -0.806368 0.810912" rpy="0 0 0"/>
+    <origin xyz="${0.176294-0.358864} ${0.41092-0.806368} ${-0.406074+0.810912}" rpy="0 0 0"/>
     <geometry>
       <mesh filename="file://$(find Dual_piper_ROS2_description)/meshes/piper_right_R_1.stl" scale="0.001 0.001 0.001"/>
@@ -378,5 +378,5 @@
   </visual>
   <collision>
-    <origin xyz="-0.358864 -0.806368 0.810912" rpy="0 0 0"/>
+    <origin xyz="${0.176294-0.358864} ${0.41092-0.806368} ${-0.406074+0.810912}" rpy="0 0 0"/>
     <geometry>
       <mesh filename="file://$(find Dual_piper_ROS2_description)/meshes/piper_right_R_1.stl" scale="0.001 0.001 0.001"/>
@@ -432,5 +432,5 @@
 </joint>
 <joint name="Slider 8" type="prismatic">
-  <origin xyz="-0.22209 0.395033 -0.406013" rpy="0 0 0"/>
+  <origin xyz="${0} ${0} ${0}" rpy="0 0 0"/>
   <parent link="piper_hand_L_1"/>
   <child link="piper_right_L_1"/>
@@ -439,5 +439,5 @@
 </joint>
 <joint name="Slider 9" type="prismatic">
-  <origin xyz="-0.22209 0.395033 -0.406013" rpy="0 0 0"/>
+  <origin xyz="${0} ${0} ${0}" rpy="0 0 0"/>
   <parent link="piper_hand_L_1"/>
   <child link="piper_left_L_1"/>
@@ -493,5 +493,5 @@
 </joint>
 <joint name="Slider 17" type="prismatic">
-  <origin xyz="0.176294 0.41092 -0.406074" rpy="0 0 0"/>
+  <origin xyz="${0} ${0} ${0}" rpy="0 0 0"/>
   <parent link="piper_hand_R_1"/>
   <child link="piper_left_R_1"/>
@@ -500,5 +500,5 @@
 </joint>
 <joint name="Slider 18" type="prismatic">
-  <origin xyz="0.176294 0.41092 -0.406074" rpy="0 0 0"/>
+  <origin xyz="${0} ${0} ${0}" rpy="0 0 0"/>
   <parent link="piper_hand_R_1"/>
   <child link="piper_right_R_1"/>
